Commit message: Added laser sensor

File: urdf/talos.xacro (robot description, xacro)
@@ -4,4 +4,7 @@
     <color rgba="0.2 0.2 0.2 1.0"/>
   </material>
+  <material name="yellow">
+    <color rgba="1 1 0 1.0"/>
+  </material>
   <gazebo reference="link_chassis">
     <material>Gazebo/DarkGrey</material>
@@ -12,4 +15,7 @@
   <gazebo reference="link_rightwheel">
     <material>Gazebo/Black</material>
+  </gazebo>
+  <gazebo reference="link_lasersensor">
+    <material>Gazebo/Yellow</material>
   </gazebo>
   <gazebo>
@@ -29,4 +35,35 @@
     </plugin>
   </gazebo>
+<gazebo reference="link_lasersensor">
+    <sensor type="ray" name="head_hokuyo_sensor">
+      <pose>0 0 0 0 0 0</pose>
+      <visualize>false</visualize>
+      <update_rate>20</update_rate>
+      <ray>
+        <scan>
+          <horizontal>
+            <samples>720</samples>
+            <resolution>1</resolution>
+            <min_angle>-1.570796</min_angle>
+            <max_angle>1.570796</max_angle>
+          </horizontal>
+        </scan>
+        <range>
+          <min>0.10</min>
+          <max>10.0</max>
+          <resolution>0.01</resolution>
+        </range>
+        <noise>
+          <type>gaussian</type>
+          <mean>0.0</mean>
+          <stddev>0.01</stddev>
+        </noise>
+      </ray>
+      <plugin name="gazebo_ros_head_hokuyo_controller" filename="libgazebo_ros_laser.so">
+        <topicName>/talos/laser/scan</topicName>
+        <frameName>link_lasersensor</frameName>
+      </plugin>
+    </sensor>
+  </gazebo>
   <link name="link_chassis">
     <!-- pose -->
@@ -39,5 +76,10 @@
       <!-- same origin as the pose-->
       <origin rpy="0 0 0" xyz="0 0 0.1"/>
-      <inertia ixx="0.0395416666667" ixy="0" ixz="0" iyy="0.106208333333" iyz="0" izz="0.106208333333"/>
+      <!-- ixx= mass*(length*length+height*height)/12
+             iyy= mass*(width*width+height*height)/12
+             izz= mass*(width*width+length*length)/12 -->
+      <inertia ixx="0.0109" ixy="0" ixz="0"
+               iyy="0.0234" iyz="0"
+               izz="0.0325"/>
     </inertial>
     <!-- body -->
@@ -79,9 +121,41 @@
     </visual>
   </link>
+<link name="link_lasersensor">
+    <inertial>
+        <origin xyz="0 0 0" rpy="0 0 0" />
+        <mass value="1" />
+        <!-- ixx= mass*(3*radius*radius+length*length)/12
+             iyy= mass*(3*radius*radius+length*length)/12
+             izz= mass*(radius*radius)/2 -->
+        <inertia  ixx="0.00013333333" ixy = "0" ixz = "0"
+            iyy="0.00013333333" iyz = "0"
+            izz="0.000125" />
+    </inertial>
+    <visual>
+        <origin xyz="0 0 0" rpy="0 0 0" />
+        <geometry>
+        <cylinder radius="0.02" length="0.02"/>
+        </geometry>
+        <material name="yellow" />
+    </visual>
+    <collision>
+        <origin xyz="0 0 0" rpy="0 0 0"/>
+        <geometry>
+        <cylinder radius="0.02" length="0.02"/>
+        </geometry>
+    </collision>
+    </link>
+    <joint name="joint_lasersensor" type="fixed">
+    <origin xyz="0.15 0 0.05" rpy="0 0 0"/>
+    <parent link="link_chassis"/>
+    <child link="link_lasersensor"/>
+  </joint>
   <link name="link_rightwheel">
     <inertial>
       <mass value="0.1"/>
       <origin rpy="0 1.5707 1.5707" xyz="0 0 0"/>
-      <inertia ixx="0.000526666666667" ixy="0" ixz="0" iyy="0.000526666666667" iyz="0" izz="0.001"/>
+      <inertia ixx="0.00006583333" ixy="0" ixz="0"
+               iyy="0.00006583333" iyz="0"
+               izz="0.000125"/>
     </inertial>
     <collision name="link_rightwheel_collision">
@@ -110,5 +184,7 @@
       <mass value="0.2"/>
       <origin rpy="0 1.5707 1.5707" xyz="0 0 0"/>
-      <inertia ixx="0.000526666666667" ixy="0" ixz="0" iyy="0.000526666666667" iyz="0" izz="0.001"/>
+      <inertia ixx="0.00006583333" ixy="0" ixz="0"
+               iyy="0.00006583333" iyz="0"
+               izz="0.001"/>
     </inertial>
     <collision name="link_leftwheel_collision">

Commit message: Added python script to read laser values

File: urdf/talos.xacro (robot description, xacro)
@@ -98,5 +98,5 @@
     <!-- thirdwheel -->
     <collision name="thirdwheel_collision">
-      <origin rpy=" 0 0 0" xyz="0.1 0 -0.03"/>
+      <origin rpy=" 0 0 0" xyz="0.15 0 -0.03"/>
       <geometry>
         <sphere radius="0.02"/>

Commit message: Changed third wheel to be more stable

File: urdf/talos.xacro (robot description, xacro)
@@ -97,5 +97,5 @@
     </visual>
     <!-- thirdwheel -->
-    <collision name="thirdwheel_collision">
+    <!--<collision name="thirdwheel_collision">
       <origin rpy=" 0 0 0" xyz="0.15 0 -0.03"/>
       <geometry>
@@ -104,7 +104,7 @@
       <surface>
         <friction>
-          <ode>
+          <ode> -->
             <!-- no friction -->
-            <mu>0</mu>
+         <!--   <mu>0</mu>
             <mu2>0</mu2>
             <slip1>1.0</slip1>
@@ -115,9 +115,34 @@
     </collision>
     <visual name="thirdwheel_visual">
-      <origin rpy=" 0 0 0" xyz="0.1 0 -0.03"/>
+      <origin rpy=" 0 0 0" xyz="0.15 0 -0.03"/>
       <geometry>
         <sphere radius="0.02"/>
       </geometry>
-    </visual>
+    </visual> -->
+  </link>
+     <!-- Caster Wheel -->
+  <joint name="fixed" type="fixed">
+    <parent link="link_chassis"/>
+    <child link="caster_wheel"/>
+  </joint>
+  <link name="caster_wheel">
+    <collision>
+      <origin rpy=" 0 0 0" xyz="-0.15 0 -0.03"/>
+      <geometry>
+    <sphere radius="0.02"/>
+      </geometry>
+    </collision>
+    <visual>
+      <origin rpy=" 0 0 0" xyz="-0.15 0 -0.03"/>
+      <geometry>
+    <sphere radius="0.02"/>
+      </geometry>
+      <material name="red"/>
+    </visual>
+    <inertia>
+      <origin xyz="-0.15 0 0.1" rpy="0 0 0"/>
+      <mass value="0.5"/>
+      <sphere_inertia m="0.5" r="0.02"/>
+    </inertia>
   </link>
 <link name="link_lasersensor">
@@ -173,5 +198,5 @@
   </link>
   <joint name="joint_rightwheel" type="continuous">
-    <origin rpy="0 0 0" xyz="-0.05 0.10 0"/>
+    <origin rpy="0 0 0" xyz="0.15 0.10 0"/>
     <child link="link_rightwheel"/>
     <parent link="link_chassis"/>
@@ -202,5 +227,5 @@
   </link>
   <joint name="joint_leftwheel" type="continuous">
-    <origin rpy="0 0 0" xyz="-0.05 -0.10 0"/>
+    <origin rpy="0 0 0" xyz="0.15 -0.10 0"/>
     <child link="link_leftwheel"/>
     <parent link="link_chassis"/>
